File: power_supply.sch (KiCad schematic (older format))
At the start: 37 parts

Commit message: Power Supply v1.0 - Gerber generated, to be manufactured
Parts:
- removed C? (x8): 1u, symbol C
- removed C? (x3): 100n, symbol C
- removed C? (x3): 1n, symbol C
- removed D? (x2): 1N4007, symbol D
- removed J?: BATTERY_A, symbol Conn_01x02
- removed J?: MASTER_JACK, symbol Conn_01x02
- removed J?: BATA_DISPLAY, symbol Conn_01x02
- removed J?: E1_JACK, symbol Conn_01x02
- removed J?: E1_OUT, symbol Conn_01x03
- removed J?: E1_BAT, symbol Conn_01x02
- removed J?: BATE1_DISPLAY, symbol Conn_01x02
- removed OK?: 4N35, DIL06, symbol 4N35
- removed Q?: IRLZ44N, TO_SOT_Packages_THT:TO-220_Vertical, symbol IRLZ44N
- removed Q? (x2): 2N7000, TO_SOT_Packages_THT:TO-92_Molded_Narrow, symbol 2N7000
- removed R?: 68K, symbol R
- removed R?: 680, symbol R
- removed R? (x3): 100, symbol R
- removed R? (x4): 47K, symbol R
- removed U?: 5V/3A, symbol 5V/3A
Connections:
- net labels removed: +5E1, GNDA, GNDE1, VBATA, VBATE1, e1_gnd, e1_jack_o, m_jack_o
- wire segments 100 -> 0
- no-connect marks 1 -> 0
Other:
- note removed: "200ms"
- note removed: "5V/3A"
- note removed: "Jack"
- note removed: "Telemetry module"
- note removed: "To be placed near load (0.78F/15V)"
- note removed: "display"
- note removed: "i_off_max = (4.2-1.1)/680 + 4.2/47k = 4.5mA\nt_2000mAh = 2000/i_off_max = 430h"
- note removed: "smooth transition in about"
- note removed: "switch inlined to"
